File: circuit_boards/base_pwr/BaSe_PWR_V4_0.kicad_pcb (KiCad board)
At the start: 2 copper layers, 78 x 65 mm, 86 parts, among them J1 12VDC In, J10 Conn_01x04_Socket, J11 Conn_01x07_Pin, J2 USB_B_Micro, J5 MOTOR, J6 USB3_B_Micro, J7 USB_C_Receptacle, J8 Screw_Terminal_01x03, J9 USB3_A, P1 USB_C_Plug, Q2 BSS214NW, Q3 BSS214NW, Q4 BSS214NW, Q5 BSS214NW, Q6 AOSP21321, U2 AMS1117-3.3, U3 STM32F070RBTx, U4 LM2596S-5, U5 DRV8220, U6 AMS1117-3.3, Y1 32.768kHz, Y2 8MHz

Commit message: BaSe PWR V4.0: split pcbs so all connectors can face far end.
Parts:
- removed C7, C8: 4.3pF, Capacitor_SMD:C_0603_1608Metric_Pad1.08x0.95mm_HandSolder
- removed J8: Screw_Terminal_01x03, TerminalBlock_Phoenix:TerminalBlock_Phoenix_MKDS-1,5-3_1x03_P5.00mm_Horizontal
- removed R4: R, Resistor_SMD:R_0603_1608Metric_Pad0.98x0.95mm_HandSolder
- removed Y1: 32.768kHz, Crystal:Crystal_SMD_Abracon_ABS25-4Pin_8.0x3.8mm
- added H1: MountingHole, MountingHole:MountingHole_2.7mm_M2.5_DIN965, F.Cu at (85.5, 142.0)
- added H2: MountingHole, MountingHole:MountingHole_2.7mm_M2.5_DIN965, F.Cu at (85.5, 129.5)
- added J12: Conn_02x06_Odd_Even, Connector_PinHeader_2.54mm:PinHeader_2x06_P2.54mm_Vertical, F.Cu at (96.0, 158.0)
- added J13: Conn_01x04_Socket, Connector_JST:JST_XH_B4B-XH-A_1x04_P2.50mm_Vertical, F.Cu at (323.0, 41.0)
- added J4: Conn_02x06_Odd_Even, Connector_PinSocket_2.54mm:PinSocket_2x06_P2.54mm_Vertical, B.Cu at (96.0, 121.5)
- added R1: 100k, Resistor_SMD:R_0603_1608Metric_Pad0.98x0.95mm_HandSolder, F.Cu at (73.0, 85.5)
- added R11: 100, Resistor_SMD:R_0603_1608Metric_Pad0.98x0.95mm_HandSolder, F.Cu at (69.6, 85.5)
- 2k10, 2k4, 2k5, 2k7, 2k8, 2k9, D10, D12, D13, D9, Q2, Q3, Q4, Q5: moved to B.Cu
- H3, H4: footprint MountingHole:MountingHole_3.2mm_M3_DIN965 -> MountingHole:MountingHole_2.7mm_M2.5_DIN965
- moved D12 140.7 mm to (79.6, 94.1), turned to 90 degrees
- moved Q5 129.7 mm to (82.6, 94.0), turned to 180 degrees
- moved C5 129.3 mm to (91.8, 78.6)
- moved C6 129.3 mm to (91.8, 71.5)
- moved R3 129.3 mm to (91.8, 75.1)
- moved D13 123.4 mm to (96.6, 94.0), turned to 90 degrees
- moved Q4 119.9 mm to (93.6, 94.0)
- moved R10 100.2 mm to (236.5, -4.99), turned to -90 degrees
- moved U6 92.2 mm to (72.0, 48.8)
- moved J11 91.8 mm to (210.4, 92.5)
- moved C19 89.1 mm to (60.0, 8.00)
- moved J5 87.9 mm to (132.8, 89.3)
- moved U5 87.9 mm to (137.8, 90.5)
- moved C22 87.9 mm to (137.7, 87.8)
- moved U2 77.1 mm to (72.0, 56.2)
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Connections:
- J10 pad 1: /+12V_sbu -> /+5V_sbu
- J10 pad 4: /+5V_sbu -> /+12V_sbu
- J7 pad A5: GND2 -> /supply_sense
- J7 pad B5: GND2 -> unconnected-(J7-CC2-PadB5)
- J7 pad B8: /supply_sense -> unconnected-(J7-SBU2-PadB8)
- P1 pad A10: +5V -> /+5V_HDD_
- P1 pad A11: +5V -> /+5V_HDD_
- P1 pad A4: +12V -> /+12V_HDD_
- P1 pad A5: GND1 -> /stator_supply_sense
- P1 pad A8: unconnected-(P1-SBU1-PadA8) -> /aux_i2c_scl
- P1 pad A9: +12V -> /+12V_HDD_
- P1 pad B2: +5V -> /+5V_HDD_
- P1 pad B3: +5V -> /+5V_HDD_
- P1 pad B4: +12V -> /+12V_HDD_
- P1 pad B5: GND1 -> /aux_3v3
- P1 pad B8: /stator_supply_docked_sense -> /aux_i2c_sda
- P1 pad B9: +12V -> /+12V_HDD_
- U3 pad 15: /stator_supply_docked_sense -> /stator_supply_sense
- U3 pad 3: Net-(U3-PC14) -> unconnected-(U3-PC14-Pad3)
- U3 pad 4: Net-(U3-PC15) -> unconnected-(U3-PC15-Pad4)
Routing:
- net /stator_d-: track 0.00 -> 27.1 mm, vias 0 -> 1
- net /stator_d+: track 0.00 -> 27.1 mm, vias 0 -> 1
- net /stator_tx-: track 0.00 -> 23.0 mm, vias 0 -> 1
- net /stator_tx+: track 0.00 -> 23.0 mm, vias 0 -> 1
- net /stator_rx-: track 0.00 -> 20.6 mm
- net /stator_rx+: track 0.00 -> 20.6 mm
Other:
- board size 78 x 65 mm -> 61.5 x 95 mm
- board text added: "Clutch"
- board text added: "Motor"
- board text added: "Spindle-Nut"

Commit message: BaSe_PWR_V4_0: add last footprints, position components
Parts:
- added C1: 4.7µF, Capacitor_THT:C_Radial_D4.0mm_H7.0mm_P1.50mm, F.Cu at (84.0, 87.5)
- added C20: 22µF, Capacitor_THT:C_Radial_D5.0mm_H11.0mm_P2.00mm, F.Cu at (66.0, 80.5)
- added C21: 22µF, Capacitor_THT:C_Radial_D5.0mm_H11.0mm_P2.00mm, F.Cu at (66.0, 73.5)
- added D11: D_Schottky, Diode_SMD:D_SOD-123, B.Cu at (79.0, 76.5)
- added D3: ~, Diode_SMD:D_SOD-123, F.Cu at (89.8, 161.5)
- added H5: MountingHole, MountingHole:MountingHole_2.7mm_M2.5_DIN965, F.Cu at (22.8, 66.2)
- added H6: MountingHole, MountingHole:MountingHole_2.7mm_M2.5_DIN965, F.Cu at (22.8, 110.8)
- added H7: MountingHole, MountingHole:MountingHole_2.7mm_M2.5_DIN965, F.Cu at (95.2, 70.0)
- added J2: ~, Connector_PinHeader_2.54mm:PinHeader_1x18_P2.54mm_Vertical, F.Cu at (53.0, 65.5)
- added R1: 100, Resistor_SMD:R_0603_1608Metric_Pad0.98x0.95mm_HandSolder, F.Cu at (70.0, 70.8)
- added R19: 100, Resistor_SMD:R_0603_1608Metric_Pad0.98x0.95mm_HandSolder, B.Cu at (78.3, 74.5)
- 2k1: renamed from 2k3; moved to B.Cu
- 2k8: renamed from 2k6; moved to B.Cu
- C10: renamed from C11; moved to B.Cu
- C16: renamed from C10; value C -> 100nF
- C17: renamed from C27; value C -> 100nF
- J12: renamed from J9; moved to B.Cu
- R2: renamed from 2k1; value ~ -> 100
- R4: renamed from R7; moved to B.Cu
- R5: renamed from R8; moved to B.Cu
- R6: renamed from R5; moved to B.Cu
- R7: renamed from R6; value 33k -> 24,9k; moved to B.Cu
- moved J8 239.9 mm to (121.0, 137.0), turned to -90 degrees
- moved J12 238.7 mm to (128.3, 133.8), turned to -90 degrees
- moved J10 224.7 mm to (123.8, 145.0)
- moved H3 219.7 mm to (118.0, 144.2)
- moved H4 209.8 mm to (118.0, 129.8)
- moved R14 204.5 mm to (123.8, 127.0), turned to 180 degrees
- moved R15 204.1 mm to (123.8, 128.5)
- moved R17 203.7 mm to (123.8, 130.0)
- moved R10 195.3 mm to (83.8, 116.8)
- moved R11 194.5 mm to (50.8, 78.4), turned to -90 degrees
- moved C18 166.3 mm to (62.5, 81.5), turned to -90 degrees
- moved R5 164.8 mm to (81.3, 82.8), turned to -90 degrees
- moved R4 163.6 mm to (82.8, 82.8), turned to -90 degrees
- moved C16 159.7 mm to (62.5, 78.1), turned to 90 degrees
- moved C8 152.4 mm to (69.6, 81.8), turned to 90 degrees
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- renumbered 2k7 to 2k2, 2k4 to 2k3, 2k8 to 2k4, 2k9 to 2k5, 2k5 to 2k6, 2k10 to 2k7, C23 to C11, C25 to C12, C26 to C13, C17 to C15, C15 to C18, C28 to C19, C5 to C2, C33 to C22, C3 to C23, C19 to C24, C22 to C25, C6 to C3, C9 to C4, C1 to C5, C12 to C6, C2 to C7, C13 to C8, C16 to C9, D8 to D10, D5 to D2, D9 to D4, D12 to D5, D10 to D6, D13 to D7, D6 to D8, D7 to D9, J13 to J10, J5 to J11, J2 to J3, J11 to J4, J4 to J5, J12 to J7, J7 to J8, J10 to J9, Q6 to Q1, Q3 to Q2, Q5 to Q3, Q2 to Q5, R9 to R11, R17 to R14, R18 to R15, R14 to R16, R19 to R17, R15 to R18, R11 to R8, R1 to R9, U3 to U1, U4 to U2, U2 to U3, U6 to U4, Y2 to Y1
Connections:
- C10 pad 1: /12vin_meas -> Net-(D11-K)
- R6 pad 1: /12vin_meas -> Net-(D11-K)
- R7 pad 2: /12vin_meas -> Net-(D11-K)
- U1 pad 20: unconnected-(U3-PA4-Pad20) -> /12vin_meas
- U1 pad 26: /Dis_PWM -> /hmi_pwm0
Routing:
- net /stator_d-: track 27.1 -> 31.9 mm
- net /stator_d+: track 27.1 -> 31.9 mm
- net /stator_tx-: track 23.0 -> 27.7 mm
- net /stator_rx-: track 20.6 -> 25.3 mm
- net /stator_rx+: track 20.6 -> 25.3 mm
- net /stator_tx+: track 23.0 -> 27.7 mm
Other:
- board size 61.5 x 95 mm -> 114.2 x 103.5 mm

Commit message: BaSe PWR V4.0: add stub for power backup based on 9V block
Parts:
- added C26: 10µF, Capacitor_SMD:C_1206_3216Metric_Pad1.33x1.80mm_HandSolder, F.Cu at (23.8, 73.5)
- added FB1: FerriteBead, Capacitor_SMD:C_1206_3216Metric_Pad1.33x1.80mm_HandSolder, F.Cu at (21.5, 78.0)
- moved C23 0.30 mm to (25.5, 86.2)
Connections:
- C22 pad 2: +5V -> /+5v_out
- C23 pad 1: +5V -> /+5v_out
- L1 pad 2: +5V -> /+5v_out
- U2 pad 4: +5V -> /+5v_out
