File: circuit_boards/base_pwr/BaSe_PWR_V4_0.kicad_sch (KiCad schematic)
At the start: 17 parts, among them J1 USB_B, J2 MOTOR, J3 MEAS, J4 USB_B_Micro, J5 Conn_02x19_Odd_Even, U1 DRV8220, U2 STM32F070CBTx

Commit message: base_pwr: rescure schematic parts from old version (v3.2) and start with mcu wiring
Parts:
- removed J1: USB_B, Connector_USB:USB_B_Lumberg_2411_02_Horizontal, symbol Connector:USB_B
- removed J3: MEAS, Connector_PinHeader_2.54mm:PinHeader_1x02_P2.54mm_Vertical, symbol Connector:Conn_01x02_Female
- removed J5: Conn_02x19_Odd_Even, Connector_PinHeader_2.54mm:PinHeader_2x19_P2.54mm_Vertical, symbol Connector_Generic:Conn_02x19_Odd_Even
- removed U2: STM32F070CBTx, Package_QFP:LQFP-48_7x7mm_P0.5mm, symbol MCU_ST_STM32F0:STM32F070CBTx
- added 2k2, 2k3, 2k4, 2k5, 2k6, 2k8, R11, R15: ~, Resistor_SMD:R_0603_1608Metric_Pad0.98x0.95mm_HandSolder, symbol BackupServer-rescue:R-BackupServer-rescue
- added C10: C, Capacitor_SMD:C_0603_1608Metric_Pad1.08x0.95mm_HandSolder, symbol Device:C
- added C12, C13, C15, C16, C9: 100nF, Capacitor_SMD:C_0603_1608Metric_Pad1.08x0.95mm_HandSolder, symbol Device:C
- added C12, C15: ~, Capacitor_SMD:C_0603_1608Metric_Pad1.08x0.95mm_HandSolder, symbol BackupServer-rescue:C-BackupServer-rescue
- added C14: ~, Capacitor_SMD:C_0603_1608Metric_Pad1.08x0.95mm_HandSolder, symbol Waberinator_rev1-rescue:CP
- added C17, C2, C20, C3: ~, Capacitor_SMD:C_0603_1608Metric_Pad1.08x0.95mm_HandSolder, symbol Device:C_Small
- added C17: ~, Capacitor_SMD:C_0603_1608Metric_Pad1.08x0.95mm_HandSolder, symbol Waberinator_rev1-rescue:C
- added C18: 22µF, symbol Device:C
- added C5, C6: 20pF, Capacitor_SMD:C_0603_1608Metric_Pad1.08x0.95mm_HandSolder, symbol Device:C
- added C6: 100nF, Capacitor_SMD:C_0603_1608Metric_Pad1.08x0.95mm_HandSolder, symbol Waberinator_rev1-rescue:C
- added C7, C8: 4.3pF, Capacitor_SMD:C_0603_1608Metric_Pad1.08x0.95mm_HandSolder, symbol Device:C
- added D10, D9: ~, symbol BackupServer-rescue:D-BackupServer-rescue
- added D3: ~, symbol Device:D_TVS
- added D4, D5: ~, symbol Device:D_Zener
- added D5: SK34-TP, Diode_SMD:D_SMC_Handsoldering, symbol Device:D_Schottky
- added D6: ~, symbol Device:D_Schottky
- added F1: ~, symbol Device:Fuse
- added FFC_Cable1: ~, symbol Connector:Conn_01x01_Female
- added FL1, FL2: ~, symbol Device:EMI_Filter_LL_1423
- added H1, H2, H3, H4: MountingHole, MountingHole:MountingHole_3.2mm_M3_DIN965, symbol Mechanical:MountingHole
- added J1: 12VDC In, symbol Connector:Conn_01x02_Pin
- added J1: USB_C_Receptacle, g7_connectors:conn_usbc_socket_RAHPCUC31AU1TR, symbol Connector:USB_C_Receptacle
- added J2: ~, symbol Connector_Generic:Conn_01x02
- added J3: USB3_A, g7_connectors:STEWARD_USB3_A_SS-52000-001, symbol Connector:USB3_A
- added J5: ~, symbol Connector:Conn_01x18_Female
- added J5: Screw_Terminal_01x03, TerminalBlock_Phoenix:TerminalBlock_Phoenix_MKDS-1,5-3_1x03_P5.00mm_Horizontal, symbol Connector:Screw_Terminal_01x03
- added J7: USB3_B_Micro, g7_connectors:conn_usb3bmicro_GSB343K331HR, symbol Connector:USB3_B_Micro
- added K1: ~, symbol g7_custom:EC2-12TNU
- added L1: 47µH, Inductor_SMD:L_Wuerth_WE-PD-Typ-LS_Handsoldering, symbol Device:L
- added P1: USB_C_Plug, g7_connectors:Molex_USBC_Plug_1054440011, symbol Connector:USB_C_Plug
- added Q2: ~, symbol Transistor_FET:BSS123
- added Q3: ~, symbol Transistor_FET:BSC028N06LS3
- added Q4, Q5: BS170, symbol Transistor_FET:BS170
- added Q4: ~, symbol g7_custom:BSC093N04LS
- added R1: 31k6, Resistor_SMD:R_0603_1608Metric_Pad0.98x0.95mm_HandSolder, symbol Device:R
- added R2: 38k3, Resistor_SMD:R_0603_1608Metric_Pad0.98x0.95mm_HandSolder, symbol Device:R
- added R3, R7, R8: 10k, Resistor_SMD:R_0603_1608Metric_Pad0.98x0.95mm_HandSolder, symbol Device:R
- added R3: ~, Resistor_SMD:R_0603_1608Metric_Pad0.98x0.95mm_HandSolder, symbol Device:R_Small
- added R3, R4 (x2): R, Resistor_SMD:R_0603_1608Metric_Pad0.98x0.95mm_HandSolder, symbol Device:R
- added R6: 100k, Resistor_SMD:R_0603_1608Metric_Pad0.98x0.95mm_HandSolder, symbol Waberinator_rev1-rescue:R
- added R7: 33k, Resistor_SMD:R_0603_1608Metric_Pad0.98x0.95mm_HandSolder, symbol Waberinator_rev1-rescue:R
- added R9: 47k, Resistor_SMD:R_0603_1608Metric_Pad0.98x0.95mm_HandSolder, symbol Device:R
- added TP1: TestPoint, symbol Connector:TestPoint
- added U2: AMS1117-3.3, Package_TO_SOT_SMD:SOT-223-3_TabPin2, symbol Regulator_Linear:AMS1117-3.3
- added U3: STM32F070RBTx, Package_QFP:LQFP-64_10x10mm_P0.5mm, symbol MCU_ST_STM32F0:STM32F070RBTx
- added U4: LM2596S-5, Package_TO_SOT_SMD:TO-263-5_TabPin3, symbol Regulator_Switching:LM2596S-5
- added U4: ~, symbol Power_Management:LTC4359-MS8
- added Y1: 32.768kHz, Crystal:Crystal_SMD_Abracon_ABS25-4Pin_8.0x3.8mm, symbol Device:Crystal
- added Y2: 8MHz, Crystal:Crystal_SMD_HC49-SD_HandSoldering, symbol Device:Crystal
- J2: renamed from J4; footprint (none) -> Connector_USB:USB_Micro-B_Molex-105017-0001
- R10: renamed from R5; footprint (none) -> Resistor_SMD:R_0603_1608Metric_Pad0.98x0.95mm_HandSolder
- renumbered C1 to C19, C2 to C22, D1 to D6, D2 to D7, D3 to D8, J2 to J5, R1 to R12, R2 to R13, R3 to R14, R4 to R15, U1 to U5
Connections:
- net GND: now also 2k4.1, 2k5.1, C10.2, C12.2, C13.2, C14.2, C15.2, C15.2, C16.2, C17.1, C17.2, C18.2, C3.2, C5.1, C6.1, C6.2, C7.1, C8.1, C9.2, D3.2 (A2), D5.2 (A), FL1.3, FL2.4, J5.13 (Pin_13), J5.14 (Pin_14), J5.15 (Pin_15), J5.16 (Pin_16), J5.7 (Pin_7), J5.8 (Pin_8), K1.10, K1.3, Q2.2 (S), Q4.3 (S), Q5.3 (S), R3.2, R7.1, R8.2, U2.1 (GND), U4.3 (GND)
- net USB_DM: now also U3.44 (PA11)
- net USB_DP: now also U3.45 (PA12)
- net imotor: now also TP1.1
- net imotor_prot: now also U3.14 (PA0)
- net vbus_sense: now also U3.42 (PA9)
- net Vdrive renamed +12V
- net +12V: now also C10.1, C12.1, C14.1, C15.1, C17.2, D10.1 (K), D6.1 (K), D9.1 (K), K1.1, K1.6, K1.8, P1.A4 (VBUS), P1.A9 (VBUS), P1.B4 (VBUS), P1.B9 (VBUS), Q3.5 (D), R11.1, R6.2, U2.3 (VI), U4.1 (VIN), U4.8 (OUT)
- new net: J7.1 (VBUS), R4.1
- new net: C17.1, FL2.3, Q4.1 (S), Q4.2 (S), Q4.3 (S)
- new net: R15.2, U4.5 (~{SHDN})
- new net: C7.2, R4.1, U3.3 (PC14), Y1.2
- new net: C8.2, R4.2, U3.4 (PC15), Y1.1
- new net: C20.2, FL2.1, J2.1 (Pin_1)
- new net: C20.1, FL2.2, J2.2 (Pin_2)
- new net: 2k3.2, 2k4.2, Q4.2 (G)
- new net: C12.2, D5.1 (K), R3.1, U4.6 (Vss)
- new net: D4.2 (A), D5.2 (A)
- new net: D9.2 (A), K1.12, Q4.1 (D)
- new net: D10.2 (A), K1.7, Q5.1 (D)
- new net: C5.2, R3.1, U3.5 (PF0), Y2.2
- new net: C6.2, R3.2, U3.6 (PF1), Y2.1
- new net: 2k5.2, 2k6.2, Q5.2 (G)
- new net: C3.1, F1.2, FL1.4
- new net: Q3.4 (G), U4.1 (GATE)
- new net: Q2.3 (D), Q4.4 (G), R11.2
- new net: U3.18 (VSS), U3.31 (VSS), U3.47 (VSS), U3.63 (VSS)
- new net +12VA: J1.A4 (VBUS), J1.A9 (VBUS), J1.B4 (VBUS), J1.B9 (VBUS), J5.1 (Pin_1), R2.1
- new net +12V_HDD: K1.9
- new net +3V3_STBY: 2k2.2, C12.1, C13.1, C15.1, C16.1, C18.1, C9.1, R7.2, R9.1, U2.2 (VO), U3.1 (VDD), U3.13 (VDDA), U3.19 (VDD), U3.32 (VDD), U3.48 (VDD), U3.64 (VDD)
- new net +5V: J5.10 (Pin_10), J5.9 (Pin_9), K1.5, L1.2, P1.A10 (RX2-), P1.A11 (RX2+), P1.B2 (TX2+), P1.B3 (TX2-), Q4.5 (D), U4.4 (FB)
- new net +5VA: J1.A10 (RX2-), J1.A11 (RX2+), J1.B2 (TX2+), J1.B3 (TX2-), J3.1 (VBUS), J5.2 (Pin_2), R1.1
- new net +5V_HDD: K1.4
- new net 12V_nProt: D3.1 (A1), D4.1 (K), D6.2 (A), F1.1, Q3.1 (S), Q3.2 (S), Q3.3 (S), R15.1, U4.2 (SRC), U4.4 (IN)
- new net DC_IN+: C2.2, FL1.1, J1.1 (Pin_1)
- new net DC_IN-: C2.1, FL1.2, J1.2 (Pin_2)
- new net DIS_BPi_SPLY: 2k2.1, Q2.1 (G)
- new net Dis_DB4: J5.4 (Pin_4)
- new net Dis_DB5: J5.3 (Pin_3)
- new net Dis_DB6: J5.2 (Pin_2)
- new net Dis_DB7: J5.1 (Pin_1)
- new net Dis_E: J5.5 (Pin_5)
- new net Dis_PWM: J5.12 (Pin_12)
- new net Dis_RS: J5.6 (Pin_6)
- new net GND1: J7.11 (SHIELD), J7.5 (GND), J7.8 (DRAIN), P1.A1 (GND), P1.A12 (GND), P1.A5 (CC), P1.B1 (GND), P1.B12 (GND), P1.B5 (VCONN), P1.S1 (SHIELD)
- new net GND2: J1.A1 (GND), J1.A12 (GND), J1.A5 (CC1), J1.B1 (GND), J1.B12 (GND), J1.B5 (CC2), J1.S1 (SHIELD), J3.10 (SHIELD), J3.4 (GND), J3.7 (DRAIN), J5.3 (Pin_3), R3.2
- new net LED_HMI: 2k8.2, J5.11 (Pin_11)
- new net LED_HMI_attiny: 2k8.1
- new net SW: D5.1 (K), L1.1, U4.2 (OUT)
- new net SW_HDD_Off: 2k6.1
- new net SW_HDD_On: 2k3.1
- new net Taster_0: J5.17 (Pin_17)
- new net Taster_1: J5.18 (Pin_18)
- new net adc_vbat: C6.1, R6.1, R7.2
- new net boot0: R8.1, U3.60 (BOOT0)
- new net hmi_miso2_sda2: U3.35 (PB14)
- new net hmi_mosi2: U3.36 (PB15)
- new net hmi_nss2: U3.33 (PB12)
- new net hmi_pushbutton_0: U3.28 (PB2)
- new net hmi_pushbutton_1: U3.55 (PB3)
- new net hmi_pwm0: U3.26 (PB0)
- new net hmi_pwm1: U3.27 (PB1)
- new net hmi_sck2_scl2: U3.34 (PB13)
- new net hmi_usart_rx3: U3.30 (PB11)
- new net hmi_usart_tx3: U3.29 (PB10)
- new net l1_rx+: J1.B11 (RX1+), J3.6 (SSRX+)
- new net l1_rx-: J1.B10 (RX1-), J3.5 (SSRX-)
- new net l1_tx+: J1.A2 (TX1+), J3.9 (SSTX+)
- new net l1_tx-: J1.A3 (TX1-), J3.8 (SSTX-)
- new net lane1_d+: J1.A6 (D+), J3.3 (D+)
- new net lane1_d-: J1.A7 (D-), J3.2 (D-)
- new net stator_d+: J7.3 (D+), P1.A6 (D+)
- new net stator_d-: J7.2 (D-), P1.A7 (D-)
- new net stator_rx+: J7.10 (SSRX+), P1.B11 (RX1+)
- new net stator_rx-: J7.9 (SSRX-), P1.B10 (RX1-)
- new net stator_supply_docked_sense: P1.B8 (SBU2), U3.15 (PA1)
- new net stator_tx+: J7.7 (SSTX+), P1.A2 (TX1+)
- new net stator_tx-: J7.6 (SSTX-), P1.A3 (TX1-)
- new net supply_sense: J1.B8 (SBU2), R1.2, R2.2, R3.1
- new net ~{LM2596S_ON}: R9.2, U4.5 (~{ON}/OFF)
- new net ~{rst}: R7.1, U3.7 (NRST)
- no-connect marks 0 -> 3
Other:
- note added: "(R25 fitted) if DIS_BPi_SLPY = HiZ: Q2 Opens Q4 conducts 5V is passed to BPi"
- note added: "12V 5V V(supply_sense) ------------------------ 0 0 0V 0 1 1V 1 0 2V 1 1 3V"
- note added: "ADC_IN0"
- note added: "ADC_IN1"
- note added: "BaSe Carriage PCB"
- note added: "BaSe Static PCB"
- note added: "Operating: 4V - 80V Withstands: -40V - 100V"
- note added: "Pins betwenn HMI and PWR are crossed (1 <-> 18 etc)"
- note added: "TIM3_CH3"
- note added: "TIM3_CH4"
- note added: "auf J5 des BPi"
- note added: "docked_sense SBU1 has a pullup on the mcu-side SBU1 will go low when docked"
- note added: "for reference"
- note added: "fsw = 500kHz"
- note added: "polarity checked"
- moved on the sheet: C19, C22, D6, D7, D8, J2, J5, R10, R12, R13, R14, R15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

Commit message: BaSe_PWR_V4_0: wire up things
Parts:
- removed 2k2, R11: ~, Resistor_SMD:R_0603_1608Metric_Pad0.98x0.95mm_HandSolder, symbol BackupServer-rescue:R-BackupServer-rescue
- removed C6: 100nF, Capacitor_SMD:C_0603_1608Metric_Pad1.08x0.95mm_HandSolder, symbol Waberinator_rev1-rescue:C
- removed H3, H4: MountingHole, MountingHole:MountingHole_3.2mm_M3_DIN965, symbol Mechanical:MountingHole
- removed J2: ~, symbol Connector_Generic:Conn_01x02
- removed Q2: ~, symbol Transistor_FET:BSS123
- removed Q4, Q5: BS170, symbol Transistor_FET:BS170
- removed Q4: ~, symbol g7_custom:BSC093N04LS
- removed R4: R, Resistor_SMD:R_0603_1608Metric_Pad0.98x0.95mm_HandSolder, symbol Device:R
- removed R7: 33k, Resistor_SMD:R_0603_1608Metric_Pad0.98x0.95mm_HandSolder, symbol Waberinator_rev1-rescue:R
- added 2k10, 2k7, 2k8, 2k9: ~, Resistor_SMD:R_0603_1608Metric_Pad0.98x0.95mm_HandSolder, symbol BackupServer-rescue:R-BackupServer-rescue
- added C11: 100nF, Capacitor_SMD:C_0603_1608Metric_Pad1.08x0.95mm_HandSolder, symbol Waberinator_rev1-rescue:C
- added C23, C28: 100nF, Capacitor_SMD:C_0603_1608Metric_Pad1.08x0.95mm_HandSolder, symbol Device:C
- added C24: 4.7µF, symbol Device:C
- added C25: 10nF, Capacitor_SMD:C_0603_1608Metric_Pad1.08x0.95mm_HandSolder, symbol Device:C
- added C26: 1µF, Capacitor_SMD:C_0603_1608Metric_Pad1.08x0.95mm_HandSolder, symbol Device:C
- added C27: C, Capacitor_SMD:C_0603_1608Metric_Pad1.08x0.95mm_HandSolder, symbol Device:C
- added C29: 22µF, symbol Device:C
- added C30, C31: ~, Capacitor_SMD:C_0603_1608Metric_Pad1.08x0.95mm_HandSolder, symbol Device:C_Small
- added D11: ~, symbol Device:D_Schottky
- added D12, D13: ~, Diode_SMD:D_SOD-123F, symbol BackupServer-rescue:D-BackupServer-rescue
- added FL3: ~, g7_emi:CMC_Laird_CM2021Y330R-10, symbol Device:EMI_Filter_LL_1423
- added J11: Conn_01x07_Pin, symbol Connector:Conn_01x07_Pin
- added J4: Screw_Terminal_01x04, TerminalBlock_Phoenix:TerminalBlock_Phoenix_MKDS-1,5-4_1x04_P5.00mm_Horizontal, symbol Connector:Screw_Terminal_01x04
- added K2: ~, g7_relay:Kemet_EC2-12TNU, symbol g7_custom:EC2-12TNU
- added Q2, Q3, Q4, Q5: BSS214NW, Package_TO_SOT_SMD:SOT-323_SC-70, symbol Transistor_FET:BSS214NW
- added R5: 100k, Resistor_SMD:R_0603_1608Metric_Pad0.98x0.95mm_HandSolder, symbol Waberinator_rev1-rescue:R
- added U6: AMS1117-3.3, Package_TO_SOT_SMD:SOT-223-3_TabPin2, symbol Regulator_Linear:AMS1117-3.3
- D10, D9: footprint (none) -> Diode_SMD:D_SOD-123F
- D4: renamed from D6; now not fitted
- FL1, FL2: footprint (none) -> g7_emi:CMC_Laird_CM2021Y330R-10
- K1: footprint (none) -> g7_relay:Kemet_EC2-12TNU
- R6: value 100k -> 33k
- renumbered 2k8 to 2k1, C2 to C1, C3 to C2, C17 to C20, C20 to C21, C12 to C3, C15 to C4, D3 to D1, D4 to D2, D5 to D3, J5 to J3, Q3 to Q1, R15 to R1, R3 to R2, U4 to U1
Connections:
- net LED_HMI_attiny is gone; now on net hmi_pwm1: 2k1.1
- net adc_vbat is gone; now on net GND: R6.1
- net hmi_miso2_sda2 is gone; now on net Dis_DB6: U3.35 (PB14)
- net hmi_mosi2 is gone; now on net Dis_DB7: U3.36 (PB15)
- net hmi_nss2 is gone; now on net Dis_DB4: U3.33 (PB12)
- net hmi_pwm0 is gone; now on net Dis_PWM: U3.26 (PB0)
- net hmi_sck2_scl2 is gone; now on net Dis_DB5: U3.34 (PB13)
- net hmi_usart_rx3 is gone; now on net Dis_E: U3.30 (PB11)
- net hmi_usart_tx3 is gone; now on net Dis_RS: U3.29 (PB10)
- net +12V: now also C27.1, D12.1 (K), D13.1 (K), K2.1, K2.6, K2.8, U6.3 (VI); no longer R6.2
- net +12V_HDD: now also K2.9; no longer K1.9
- net +3V3_STBY: now also C23.1, C24.1, J11.1 (Pin_1); no longer U3.13 (VDDA)
- net +5V: now also D11.1 (K), K2.5
- net +5V_HDD: now also K2.4; no longer K1.4
- net 12V_nProt: now also R5.2
- net GND: now also U3.12 (VSSA), U3.18 (VSS), U3.31 (VSS), U3.47 (VSS), U3.63 (VSS), 2k8.1, 2k9.1, C11.2, C23.2, C24.2, C25.2, C26.2, C27.2, C28.2, C29.2, C30.2, FL3.4, K2.10, K2.3, Q2.2 (S), Q3.2 (S), Q4.2 (S), Q5.2 (S), U6.1 (GND)
- net GND1: now also J11.3 (Pin_3)
- net SW_HDD_Off: now also U3.9 (PC1), 2k10.1; no longer 2k6.1
- net SW_HDD_On: now also U3.8 (PC0), 2k7.1; no longer 2k3.1
- net Taster_0: now also U3.25 (PC5)
- net Taster_1: now also U3.37 (PC6)
- net in1_mcu: now also U3.41 (PA8)
- net in2_mcu: now also U3.23 (PA7)
- net ~{LM2596S_ON}: now also U3.24 (PC4)
- net ~{rst}: now also J11.5 (Pin_5)
- net at J7.1 (VBUS): now also D11.2 (A)
- net +5V_sbu: now reaches C20.1, FL2.3
- net +5V_sbu: now also K1.4
- net +5v_sbu_flt_gnd: now reaches C21.2, FL2.1
- net +5v_sbu_flt_gnd: now also J4.3 (Pin_3)
- net +5v_sbu_flt: now reaches C21.1, FL2.2
- net +5v_sbu_flt: now also J4.4 (Pin_4)
- net at 2k3.2, 2k4.2: now also Q3.1 (G)
- net at D9.2 (A), K1.12: now also Q3.3 (D)
- net at D10.2 (A), K1.7: now also Q2.3 (D)
- net at 2k5.2, 2k6.2: now also Q2.1 (G)
- net sw_sbu_on: now reaches U3.10 (PC2)
- net sw_sbu_on: now also 2k3.1
- net sw_sbu_off: now reaches U3.11 (PC3)
- net sw_sbu_off: now also 2k6.1
- net usart2_tx: now reaches U3.16 (PA2)
- net usart2_rx: now reaches U3.17 (PA3)
- net swdio: now reaches U3.46 (PA13)
- net swdio: now also J11.4 (Pin_4)
- net swclk: now reaches U3.49 (PA14)
- net swclk: now also J11.2 (Pin_2)
- net spi1_nss: now reaches U3.50 (PA15)
- net spi1_cipo: now reaches U3.56 (PB4)
- net spi1_copi: now reaches U3.57 (PB5)
- net usart1_tx: now reaches U3.58 (PB6)
- net usart1_tx: now also J11.6 (Pin_6)
- net usart1_rx: now reaches U3.59 (PB7)
- net usart1_rx: now also J11.7 (Pin_7)
- net i2c1_scl: now reaches U3.61 (PB8)
- net i2c1_sda: now reaches U3.62 (PB9)
- net hmi_pushbutton_0: no longer names the net of U3.28 (PB2)
- net hmi_pushbutton_1 renamed spi1_sck
- new net: D13.2 (A), K2.7, Q4.3 (D)
- new net: 2k7.2, 2k8.2, Q5.1 (G)
- new net: D12.2 (A), K2.12, Q5.3 (D)
- new net: 2k10.2, 2k9.2, Q4.1 (G)
- new net +12V_sbu: C30.1, FL3.3, K1.9
- new net +12v_sbu_flt: C31.1, FL3.2, J4.1 (Pin_1)
- new net +12v_sbu_flt_gnd: C31.2, FL3.1, J4.2 (Pin_2)
- new net +3.3VA: C25.1, C26.1, C28.1, C29.1, U3.13 (VDDA), U6.2 (VO)
- new net 12vin_meas: C11.1, R5.1, R6.2
Other:
- note added: "Pin Assignment in BaSe PWR V3.2 18: Taster_1 17: Taster_0 16-13: GND 12: Dis_PWM 11: LED_HMI 10-9: 5V 8-7: GND 6: Dis_RS 5: Dis_E 4: Dis_DB4 3: Dis_DB3 ..."
- note added: "TIM1_CH1"
- note added: "TIM1_CH1N"
- note added: "The VDDA voltage level must be always greater or equal to the VDD voltage level and must be provided first."
- note added: "power supply scheme, see datasheet section 6.1.6, p.37"
- note removed: "(R25 fitted) if DIS_BPi_SLPY = HiZ: Q2 Opens Q4 conducts 5V is passed to BPi"
- note removed: "BaSe Carriage PCB"
- note removed: "auf J5 des BPi"
- note removed: "docked_sense SBU1 has a pullup on the mcu-side SBU1 will go low when docked"
- note removed: "polarity checked"
- moved on the sheet: 2k1, 2k3, 2k4, 2k5, 2k6, C1, C10, C12, C13, C14, C15, C16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
